Commit message: feat: fixed torso joint 1

File: ros2_ws/src/galaxea_simulation/urdf/r1_v2_1_0.urdf (robot description, URDF)
Before this commit: robot r1_v2_1_0, 36 links, 35 joints
Links:
- added link base_footprint
Joints:
- added joint base_footprint_joint: type fixed, parent base_footprint, child base_link
- joint torso_joint1: axis 0 1 0 -> (none); limit lower=-1.1345 upper=1.8326 effort=100 velocity=2.5 -> (none); type revolute -> fixed

Commit message: docs: update README.md

File: ros2_ws/src/galaxea_simulation/urdf/r1_v2_1_0.urdf (robot description, URDF)
Before this commit: robot r1_v2_1_0, 37 links, 36 joints
Links:
- removed link imu_link
- removed link lidar_link
Joints:
- removed joint imu_joint
- removed joint lidar_joint
